File: pcb/pcie-mini-bridge-dev.kicad_pcb (KiCad board)
At the start: 2 copper layers, 0 parts

Commit message: dev pcb layout, outline and hole parts
Parts:
- added C1: C_Small, Capacitors_SMD:C_0603, F.Cu at (110.8, 97.2)
- added D1: Green, LEDs:LED_0603, F.Cu at (100.0, 95.2)
- added D2: Orange, LEDs:LED_0603, F.Cu at (120.2, 95.2)
- added D3: Green, LEDs:LED_0603, F.Cu at (120.2, 91.2)
- added H1: hole, pcie-mini-bridge-special:hole-m3, F.Cu at (169.7, 91.0)
- added H2: hole, pcie-mini-bridge-special:hole-m3, F.Cu at (105.3, 91.0)
- added J1: Conn_01x02, Pin_Headers:Pin_Header_Straight_1x02, F.Cu at (136.2, 91.8)
- added J2: USB_C_Receptacle, pcie-mini-bridge-special:USB_C_Receptacle_Amphenol_12401610E4-2A, F.Cu at (102.0, 104.8)
- added J3: Conn_01x02, Pin_Headers:Pin_Header_Straight_1x02, F.Cu at (131.2, 91.8)
- added J4: Conn_01x02, Pin_Headers:Pin_Header_Straight_1x02, F.Cu at (126.1, 91.8)
- added J5: PCIe_x1, pcie-mini-bridge-special:PCIe_SMDEdge_TE_5-1734857-x, F.Cu at (155.0, 90.0)
- added R1: 1k, Resistors_SMD:R_0603, F.Cu at (152.0, 97.5)
- added R10: 220, Resistors_SMD:R_0603, F.Cu at (120.2, 93.2)
- added R2: 1k, Resistors_SMD:R_0603, F.Cu at (150.0, 97.5)
- added R3: 0, Resistors_SMD:R_0603, F.Cu at (154.0, 97.5)
- added R4: 220, Resistors_SMD:R_0603, F.Cu at (100.0, 97.2)
- added R5: 27k, Resistors_SMD:R_0603, F.Cu at (110.8, 91.2)
- added R6: 10k, Resistors_SMD:R_0603, F.Cu at (110.8, 93.2)
- added R7: 27k, Resistors_SMD:R_0603, F.Cu at (110.8, 95.2)
- added R8: 220, Resistors_SMD:R_0603, F.Cu at (120.2, 97.2)
- added R9: 16.9k, Resistors_SMD:R_0603, F.Cu at (115.5, 97.2)
- added REF**: PCIe_CardOutline_x1_LPHL, pcie-mini-bridge-special:PCIe_CardOutline_x1_LPHL, F.Cu at (155.0, 87.5)
- added REF**: USB_C_PlugOutline, pcie-mini-bridge-special:USB_C_PlugOutline, F.Cu at (94.9, 104.7)
- added U1: TPS2594xx, Housings_DFN_QFN:QFN-20-1EP_3x4mm_Pitch0.5mm, F.Cu at (115.5, 93.0)
Routing:
- net GND: track 0.00 -> 131.1 mm, vias 0 -> 60
- net /PE_3V3_AUX: track 0.00 -> 83.0 mm, vias 0 -> 4
- net /PE_PRSNT2#: track 0.00 -> 74.0 mm, vias 0 -> 1
- net /PE_PRSNT1#: track 0.00 -> 72.9 mm, vias 0 -> 3
- net /PE_R0-: track 0.00 -> 67.1 mm
- net /PE_R0+: track 0.00 -> 66.5 mm
- net /PE_T0-: track 0.00 -> 63.0 mm
- net /PE_T0+: track 0.00 -> 62.4 mm
- net /PERST#: track 0.00 -> 61.4 mm, vias 0 -> 2
- net /PE_REFCLK-: track 0.00 -> 60.8 mm, vias 0 -> 1
- net /PE_REFCLK+: track 0.00 -> 60.2 mm, vias 0 -> 1
- net /BRIDGE_EN: track 0.00 -> 57.3 mm, vias 0 -> 3
- net +12V: track 0.00 -> 15.1 mm, vias 0 -> 7
- net +3V3: track 0.00 -> 15.0 mm, vias 0 -> 6
- net /PE_3V3: track 0.00 -> 9.93 mm, vias 0 -> 4
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- added copper zone on B.Cu, net +12V
- added copper zone on F.Cu, net +12V
- added copper zone on F.Cu, net +3V3
- added copper zone on In1.Cu, net +3V3
- added copper zone on B.Cu, net /PE_3V3
- added copper zone on F.Cu, net /PE_3V3
- added copper zone on B.Cu, net GND
- added copper zone on F.Cu, net GND
- added copper zone on In1.Cu, net GND
- added copper zone on In2.Cu, net GND
Other:
- board outline added: 75.4 x 23.5 mm
- copper layers 2 -> 4
- net class Default: clearance 0.2 -> 0.1524; trace_width 0.25 -> 0.2032; via_dia 0.6 -> 0.6096; via_drill 0.4 -> 0.3048
- net class PCIe Data added: clearance 0.127, trace_width 0.235, via_dia 0.7, via_drill 0.4
- rule trace_clearance: 0.2 -> 0.1524
