File: pcb/pcie-mini-bridge-host.sch (KiCad schematic (older format))
At the start: 15 parts, among them J1 PCIe_x1, J2 USB_C_Receptacle, U1 TPS25944L, U2 TPS25944L

Commit message: fix pcie footprints and remove paste and update gerbers
* fix PCIe_Fingers and PCIe_SMDEdge had bottom cu with top mask/paste
* make and use PCIe_SMDEdge-NoPaste_TE_5-1734857-x
Parts:
- D1, D2: Description (none) -> LED ORANGE CLEAR 0603 SMD; Digikey Part No (none) -> 160-1434-1-ND; Mfg (none) -> Lite-On Inc; Mfg Part No (none) -> LTST-C190KFKT
- D5: Description (none) -> LED GREEN CLEAR 0603 SMD; Digikey Part No (none) -> 160-1183-1-ND; Mfg (none) -> Lite-On Inc; Mfg Part No (none) -> LTST-C190GKT
- R10, R3, R5: value 220 -> 1k
- U1, U2: Description (none) -> IC PWR MGMT EFUSE 2.7-18V 20WQFN, Circuit Breaker, Latched; Digikey Part No (none) -> 296-42152-1-ND; Mfg (none) -> Texas Instruments; Mfg Part No (none) -> TPS25944LRVCR
Changed lines of the file:
@@
 F 2 "Housings_DFN_QFN:QFN-20-1EP_3x4mm_Pitch0.5mm" H 3400 4200 60  0001 C CNN
 F 3 "" H 3400 4200 60  0001 C CNN
+F 4 "Texas Instruments" H 3400 4300 60  0001 C CNN "Mfg"
+F 5 "TPS25944LRVCR" H 3400 4300 60  0001 C CNN "Mfg Part No"
+F 6 "296-42152-1-ND" H 3400 4300 60  0001 C CNN "Digikey Part No"
+F 7 "IC PWR MGMT EFUSE 2.7-18V 20WQFN, Circuit Breaker, Latched" H 3400 4300 60  0001 C CNN "Description"
 	1    3400 4300
 	1    0    0    -1
@@
 F 2 "Housings_DFN_QFN:QFN-20-1EP_3x4mm_Pitch0.5mm" H 3400 6400 60  0001 C CNN
 F 3 "" H 3400 6400 60  0001 C CNN
+F 4 "Texas Instruments" H 3400 6500 60  0001 C CNN "Mfg"
+F 5 "TPS25944LRVCR" H 3400 6500 60  0001 C CNN "Mfg Part No"
+F 6 "296-42152-1-ND" H 3400 6500 60  0001 C CNN "Digikey Part No"
+F 7 "IC PWR MGMT EFUSE 2.7-18V 20WQFN, Circuit Breaker, Latched" H 3400 6500 60  0001 C CNN "Description"
 	1    3400 6500
 	1    0    0    -1
@@
 P 4700 6500
 F 0 "R5" H 4730 6520 50  0000 L CNN
-F 1 "220" H 4730 6460 50  0000 L CNN
+F 1 "1k" H 4730 6460 50  0000 L CNN
 F 2 "Resistors_SMD:R_0603" H 4700 6500 50  0001 C CNN
 F 3 "" H 4700 6500 50  0001 C CNN
@@
 F 2 "LEDs:LED_0603" V 4700 6100 50  0001 C CNN
 F 3 "" V 4700 6100 50  0001 C CNN
+F 4 "Lite-On Inc" H 4700 6100 60  0001 C CNN "Mfg"
+F 5 "LTST-C190KFKT" H 4700 6100 60  0001 C CNN "Mfg Part No"
+F 6 "160-1434-1-ND" H 4700 6100 60  0001 C CNN "Digikey Part No"
+F 7 "LED ORANGE CLEAR 0603 SMD" H 4700 6100 60  0001 C CNN "Description"
 	1    4700 6100
 	0    -1   -1   0
@@
 P 4700 4300
 F 0 "R3" H 4730 4320 50  0000 L CNN
-F 1 "220" H 4730 4260 50  0000 L CNN
+F 1 "1k" H 4730 4260 50  0000 L CNN
 F 2 "Resistors_SMD:R_0603" H 4700 4300 50  0001 C CNN
 F 3 "" H 4700 4300 50  0001 C CNN
@@
 F 2 "LEDs:LED_0603" V 4700 3900 50  0001 C CNN
 F 3 "" V 4700 3900 50  0001 C CNN
+F 4 "Lite-On Inc" H 4700 3900 60  0001 C CNN "Mfg"
+F 5 "LTST-C190KFKT" H 4700 3900 60  0001 C CNN "Mfg Part No"
+F 6 "160-1434-1-ND" H 4700 3900 60  0001 C CNN "Digikey Part No"
+F 7 "LED ORANGE CLEAR 0603 SMD" H 4700 3900 60  0001 C CNN "Description"
 	1    4700 3900
 	0    -1   -1   0
@@
 P 9500 5600
 F 0 "R10" H 9530 5620 50  0000 L CNN
-F 1 "220" H 9530 5560 50  0000 L CNN
+F 1 "1k" H 9530 5560 50  0000 L CNN
 F 2 "Resistors_SMD:R_0603" H 9500 5600 50  0001 C CNN
 F 3 "" H 9500 5600 50  0001 C CNN
@@
 F 2 "LEDs:LED_0603" V 9500 5200 50  0001 C CNN
 F 3 "" V 9500 5200 50  0001 C CNN
+F 4 "Lite-On Inc" H 9500 5200 60  0001 C CNN "Mfg"
+F 5 "LTST-C190GKT" H 9500 5200 60  0001 C CNN "Mfg Part No"
+F 6 "160-1183-1-ND" H 9500 5200 60  0001 C CNN "Digikey Part No"
+F 7 "LED GREEN CLEAR 0603 SMD" H 9500 5200 60  0001 C CNN "Description"
 	1    9500 5200
 	0    -1   -1   0
